Commit message: Added all the links and joints to the robot description model

File: simulation_ws/src/manipulator_description/urdf/manipulator.xacro (robot description, xacro)
@@ -3,14 +3,14 @@
     <link name="base_link">
         <visual>
-            <origin rpy="0 0 0" xyz="0 0 0"/>
+            <origin rpy="0 0 0" xyz="0 0 0.1"/>
             <geometry>
-                <box size="1 1 1"/>
+                <box size="1 1 0.2"/>
             </geometry>
         </visual>
     </link>
-    <joint name="base_link__link_01" type="revolute">
+    <joint name="base_link__link_1" type="revolute">
         <axis xyz="0 0 1" />
         <limit effort="1000.0" lower="-3.14" upper="3.14" velocity="0.5" />
-        <origin rpy="0 0 0" xyz="0 0 0.5"/>
+        <origin rpy="0 0 0" xyz="0 0 0.2"/>
         <parent link="base_link"/>
         <child link="link1"/>
@@ -18,7 +18,37 @@
     <link name="link1">
         <visual>
-            <origin rpy="0 0 0" xyz="0 0 0.2"/>
+            <origin rpy="0 0 0" xyz="0 0 0.1"/>
             <geometry>
-                <cylinder radius="0.35" length="0.4"/>
+                <cylinder radius="0.35" length="0.2"/>
+            </geometry>
+        </visual>
+    </link>
+    <joint name="link_1__link_2" type="revolute">
+        <axis xyz="0 1 0" />
+        <limit effort="1000.0" lower="-3.14" upper="3.14" velocity="0.5" />
+        <origin rpy="0 0 0" xyz="0 0 0.2"/>
+        <parent link="link1"/>
+        <child link="link2"/>
+    </joint>
+    <link name="link2">
+        <visual>
+            <origin rpy="0 0 0" xyz="0 0 0.5"/>
+            <geometry>
+                <cylinder radius="0.15" length="1"/>
+            </geometry>
+        </visual>
+    </link>
+    <joint name="link_2__link_3" type="revolute">
+        <axis xyz="0 1 0" />
+        <limit effort="1000.0" lower="-3.14" upper="3.14" velocity="0.5" />
+        <origin rpy="0 0 0" xyz="0 0 1"/>
+        <parent link="link2"/>
+        <child link="link3"/>
+    </joint>
+    <link name="link3">
+        <visual>
+            <origin rpy="0 0 0" xyz="0 0 0.5"/>
+            <geometry>
+                <cylinder radius="0.15" length="1"/>
             </geometry>
         </visual>

Commit message: Added centralized parameters for easier configuration of the robot

File: simulation_ws/src/manipulator_description/urdf/manipulator.xacro (robot description, xacro)
@@ -1,56 +1,50 @@
 <?xml version="1.0" ?>
 <robot name="manipulator" xmlns:xacro="http://www.ros.org/wiki/xacro">
-    <link name="base_link">
-        <visual>
-            <origin rpy="0 0 0" xyz="0 0 0.1"/>
-            <geometry>
-                <box size="1 1 0.2"/>
-            </geometry>
-        </visual>
-    </link>
-    <joint name="base_link__link_1" type="revolute">
-        <axis xyz="0 0 1" />
-        <limit effort="1000.0" lower="-3.14" upper="3.14" velocity="0.5" />
-        <origin rpy="0 0 0" xyz="0 0 0.2"/>
-        <parent link="base_link"/>
-        <child link="link1"/>
-    </joint>
-    <link name="link1">
-        <visual>
-            <origin rpy="0 0 0" xyz="0 0 0.1"/>
-            <geometry>
-                <cylinder radius="0.35" length="0.2"/>
-            </geometry>
-        </visual>
-    </link>
-    <joint name="link_1__link_2" type="revolute">
-        <axis xyz="0 1 0" />
-        <limit effort="1000.0" lower="-3.14" upper="3.14" velocity="0.5" />
-        <origin rpy="0 0 0" xyz="0 0 0.2"/>
-        <parent link="link1"/>
-        <child link="link2"/>
-    </joint>
-    <link name="link2">
-        <visual>
-            <origin rpy="0 0 0" xyz="0 0 0.5"/>
-            <geometry>
-                <cylinder radius="0.15" length="1"/>
-            </geometry>
-        </visual>
-    </link>
-    <joint name="link_2__link_3" type="revolute">
-        <axis xyz="0 1 0" />
-        <limit effort="1000.0" lower="-3.14" upper="3.14" velocity="0.5" />
-        <origin rpy="0 0 0" xyz="0 0 1"/>
-        <parent link="link2"/>
-        <child link="link3"/>
-    </joint>
-    <link name="link3">
-        <visual>
-            <origin rpy="0 0 0" xyz="0 0 0.5"/>
-            <geometry>
-                <cylinder radius="0.15" length="1"/>
-            </geometry>
-        </visual>
-    </link>
+    <xacro:include filename="$(find manipulator_description)/urdf/links_joints.xacro" />
+    <xacro:include filename="$(find manipulator_description)/urdf/robot_parameters.xacro" />
+    <box_link
+      name="base_link"
+      origin_rpy="0 0 0"
+      origin_xyz="0 0 ${base_height/2}"
+      size="1 1 ${base_height}"
+    />
+    <revolute_joint
+      name="q1" type="revolute"
+      axis_xyz="0 0 1"
+      origin_rpy="0 0 0" origin_xyz="0 0 ${base_height}"
+      parent="base_link"
+      child="link1"
+      limit_e="1000.0" limit_l="-3.14" limit_u="3.14" limit_v="0.5"
+    />
+    <cylinder_link
+      name="link1"
+      origin_rpy="0 0 0" origin_xyz="0 0 ${L1/2}"
+      radius="0.35" length="${L1}"
+    />
+    <revolute_joint
+      name="q2" type="revolute"
+      axis_xyz="0 1 0"
+      origin_rpy="0 0 0" origin_xyz="0 0 ${L1}"
+      parent="link1"
+      child="link2"
+      limit_e="1000.0" limit_l="-3.14" limit_u="3.14" limit_v="0.5"
+    />
+    <cylinder_link
+      name="link2"
+      origin_rpy="0 0 0" origin_xyz="0 0 ${L2/2}"
+      radius="0.15" length="${L2}"
+    />
+    <revolute_joint
+      name="q3" type="revolute"
+      axis_xyz="0 1 0"
+      origin_rpy="0 0 0" origin_xyz="0 0 ${L2}"
+      parent="link2"
+      child="link3"
+      limit_e="1000.0" limit_l="-3.14" limit_u="3.14" limit_v="0.5"
+    />
+    <cylinder_link
+      name="link3"
+      origin_rpy="0 0 0" origin_xyz="0 0 ${L3/2}"
+      radius="0.15" length="${L3}"
+    />
 </robot>
