Commit message: dynamic model adjusted to work in Gazebo also from the same launch file

File: simulation_ws/src/manipulator_description/urdf/links_joints.xacro (robot description, xacro)
@@ -10,6 +10,11 @@
     </joint>
   </xacro:macro>
-  <xacro:macro name="cylinder_link" params="name origin_xyz origin_rpy radius length">
+  <xacro:macro name="cylinder_link" params="name origin_xyz origin_rpy radius length mass ixx ixy ixz iyy iyz izz">
     <link name="${name}">
+      <inertial>
+        <origin xyz="${origin_xyz}" rpy="${origin_rpy}"/>
+        <mass value="${mass}"/>
+        <inertia ixx="${ixx}"  ixy="${ixy}"  ixz="${ixz}" iyy="${iyy}" iyz="${iyz}" izz="${izz}" />
+      </inertial>
       <visual>
         <origin rpy="${origin_rpy}" xyz="${origin_xyz}" />
@@ -18,14 +23,31 @@
         </geometry>
       </visual>
+      <collision>
+        <origin xyz="${origin_xyz}" rpy="${origin_rpy}" />
+        <geometry>
+          <cylinder radius="${radius}" length="${length}" />
+        </geometry>
+      </collision>
     </link>
   </xacro:macro>
-  <xacro:macro name="box_link" params="name origin_xyz origin_rpy size">
+  <xacro:macro name="box_link" params="name origin_xyz origin_rpy size mass ixx ixy ixz iyy iyz izz">
     <link name="${name}">
+      <inertial>
+        <origin xyz="${origin_xyz}" rpy="${origin_rpy}"/>
+        <mass value="${mass}"/>
+        <inertia ixx="${ixx}"  ixy="${ixy}"  ixz="${ixz}" iyy="${iyy}" iyz="${iyz}" izz="${izz}" />
+      </inertial>
       <visual>
-        <origin rpy="${origin_rpy}" xyz="${origin_xyz}" />
+        <origin xyz="${origin_xyz}" rpy="${origin_rpy}" />
         <geometry>
           <box size="${size}" />
         </geometry>
       </visual>
+      <collision>
+        <origin xyz="${origin_xyz}" rpy="${origin_rpy}" />
+        <geometry>
+          <box size="${size}"/>
+        </geometry>
+      </collision>
     </link>
   </xacro:macro>

File: simulation_ws/src/manipulator_description/urdf/manipulator.xacro (robot description, xacro)
@@ -1,50 +1,72 @@
 <?xml version="1.0" ?>
 <robot name="manipulator" xmlns:xacro="http://www.ros.org/wiki/xacro">
-    <xacro:include filename="$(find manipulator_description)/urdf/links_joints.xacro" />
-    <xacro:include filename="$(find manipulator_description)/urdf/robot_parameters.xacro" />
-    <box_link
-      name="base_link"
-      origin_rpy="0 0 0"
-      origin_xyz="0 0 ${base_height/2}"
-      size="1 1 ${base_height}"
-    />
-    <revolute_joint
-      name="q1" type="revolute"
-      axis_xyz="0 0 1"
-      origin_rpy="0 0 0" origin_xyz="0 0 ${base_height}"
-      parent="base_link"
-      child="link1"
-      limit_e="1000.0" limit_l="-3.14" limit_u="3.14" limit_v="0.5"
-    />
-    <cylinder_link
-      name="link1"
-      origin_rpy="0 0 0" origin_xyz="0 0 ${L1/2}"
-      radius="0.35" length="${L1}"
-    />
-    <revolute_joint
-      name="q2" type="revolute"
-      axis_xyz="0 1 0"
-      origin_rpy="0 0 0" origin_xyz="0 0 ${L1}"
-      parent="link1"
-      child="link2"
-      limit_e="1000.0" limit_l="-3.14" limit_u="3.14" limit_v="0.5"
-    />
-    <cylinder_link
-      name="link2"
-      origin_rpy="0 0 0" origin_xyz="0 0 ${L2/2}"
-      radius="0.15" length="${L2}"
-    />
-    <revolute_joint
-      name="q3" type="revolute"
-      axis_xyz="0 1 0"
-      origin_rpy="0 0 0" origin_xyz="0 0 ${L2}"
-      parent="link2"
-      child="link3"
-      limit_e="1000.0" limit_l="-3.14" limit_u="3.14" limit_v="0.5"
-    />
-    <cylinder_link
-      name="link3"
-      origin_rpy="0 0 0" origin_xyz="0 0 ${L3/2}"
-      radius="0.15" length="${L3}"
-    />
+  <!-- Include xacros that define the types of joints and links present -->
+  <xacro:include filename="$(find manipulator_description)/urdf/links_joints.xacro" />
+  <!-- Constant definitions -->
+  <xacro:property name="base_height" value="0.2" />
+  <xacro:property name="L1" value="0.2" />
+  <xacro:property name="L2" value="1.2" />
+  <xacro:property name="L3" value="1.6" />
+  <!-- Definition of the robot using the included macros -->
+  <box_link
+    name = "base_link"
+    origin_rpy = "0 0 0"
+    origin_xyz = "0 0 ${base_height/2}"
+    size = "1 1 ${base_height}"
+    mass = "10"
+    ixx = "10" ixy = "0"   ixz = "0"
+               iyy = "10"  iyz = "0"
+                           izz = "10"
+  />
+  <revolute_joint
+    name="q1" type="revolute"
+    axis_xyz="0 0 1"
+    origin_rpy="0 0 0" origin_xyz="0 0 ${base_height}"
+    parent="base_link"
+    child="link1"
+    limit_e="1000.0" limit_l="-3.14" limit_u="3.14" limit_v="0.5"
+  />
+  <cylinder_link
+    name="link1"
+    origin_rpy="0 0 0" origin_xyz="0 0 ${L1/2}"
+    radius="0.35" length="${L1}"
+    mass = "4"
+    ixx = "3" ixy = "0"   ixz = "0"
+              iyy = "3"  iyz = "0"
+                          izz = "3"
+  />
+  <revolute_joint
+    name="q2" type="revolute"
+    axis_xyz="0 1 0"
+    origin_rpy="0 0 0" origin_xyz="0 0 ${L1}"
+    parent="link1"
+    child="link2"
+    limit_e="1000.0" limit_l="-3.14" limit_u="3.14" limit_v="0.5"
+  />
+  <cylinder_link
+    name="link2"
+    origin_rpy="0 0 0" origin_xyz="0 0 ${L2/2}"
+    radius="0.15" length="${L2}"
+    mass = "6"
+    ixx = "5" ixy = "0"   ixz = "0"
+              iyy = "5"  iyz = "0"
+                          izz = "5"
+  />
+  <revolute_joint
+    name="q3" type="revolute"
+    axis_xyz="0 1 0"
+    origin_rpy="0 0 0" origin_xyz="0 0 ${L2}"
+    parent="link2"
+    child="link3"
+    limit_e="1000.0" limit_l="-3.14" limit_u="3.14" limit_v="0.5"
+  />
+  <cylinder_link
+    name="link3"
+    origin_rpy="0 0 0" origin_xyz="0 0 ${L3/2}"
+    radius="0.15" length="${L3}"
+    mass = "8"
+    ixx = "6" ixy = "0"   ixz = "0"
+              iyy = "6"   iyz = "0"
+                          izz = "6"
+  />
 </robot>

Commit message: fixed robot to ground, added transmissions to the model as well as PID position controller to all the joints

File: simulation_ws/src/manipulator_description/urdf/links_joints.xacro (robot description, xacro)
@@ -1,4 +1,5 @@
 <?xml version="1.0" ?>
 <robot xmlns:xacro="http://www.ros.org/wiki/xacro">
+  <!-- Joint macro definitions -->
   <xacro:macro name="revolute_joint" params="name type axis_xyz origin_rpy origin_xyz parent child limit_e limit_l limit_u limit_v">
     <joint name="${name}" type="${type}">
@@ -9,5 +10,17 @@
       <child link="${child}" />
     </joint>
+    <transmission name = "${name}_trans">
+      <type>transmission_interface/SimpleTransmission</type>
+      <joint name = "${name}">
+        <hardwareInterface>hardware_interface/EffortJointInterface</hardwareInterface>
+      </joint>
+      <actuator name = "${name}_motor">
+        <mechanicalReduction> 1 </mechanicalReduction>
+        <hardwareInterface>hardware_interface/EffortJointInterface</hardwareInterface>
+      </actuator>
+    </transmission>
   </xacro:macro>
+  <!-- End joint macro definitions -->
+  <!-- Link macro definitions -->
   <xacro:macro name="cylinder_link" params="name origin_xyz origin_rpy radius length mass ixx ixy ixz iyy iyz izz">
     <link name="${name}">
@@ -52,3 +65,4 @@
     </link>
   </xacro:macro>
+  <!-- End link macro definitions -->
 </robot>

File: simulation_ws/src/manipulator_description/urdf/manipulator.xacro (robot description, xacro)
@@ -1,12 +1,18 @@
-<?xml version="1.0" ?>
-<robot name="manipulator" xmlns:xacro="http://www.ros.org/wiki/xacro">
+<?xml version = "1.0" ?>
+<robot name = "manipulator" xmlns:xacro="http://www.ros.org/wiki/xacro">
   <!-- Include xacros that define the types of joints and links present -->
-  <xacro:include filename="$(find manipulator_description)/urdf/links_joints.xacro" />
+  <xacro:include filename = "$(find manipulator_description)/urdf/links_joints.xacro" />
   <!-- Constant definitions -->
-  <xacro:property name="base_height" value="0.2" />
-  <xacro:property name="L1" value="0.2" />
-  <xacro:property name="L2" value="1.2" />
-  <xacro:property name="L3" value="1.6" />
+  <xacro:property name = "base_height" value = "0.2" />
+  <xacro:property name = "L1" value = "0.2" />
+  <xacro:property name = "L2" value = "1.2" />
+  <xacro:property name = "L3" value = "1.6" />
   <!-- Definition of the robot using the included macros -->
+  <!-- Used for fixing robot to Gazebo 'base_link' -->
+  <link name="world"/>
+  <joint name="fixed" type="fixed">
+    <parent link="world"/>
+    <child link="base_link"/>
+  </joint>
   <box_link
     name = "base_link"
@@ -20,15 +26,15 @@
   />
   <revolute_joint
-    name="q1" type="revolute"
-    axis_xyz="0 0 1"
-    origin_rpy="0 0 0" origin_xyz="0 0 ${base_height}"
-    parent="base_link"
-    child="link1"
-    limit_e="1000.0" limit_l="-3.14" limit_u="3.14" limit_v="0.5"
+    name = "q1" type = "revolute"
+    axis_xyz = "0 0 1"
+    origin_rpy = "0 0 0" origin_xyz = "0 0 ${base_height}"
+    parent = "base_link"
+    child = "link1"
+    limit_e = "1000.0" limit_l = "-3.14" limit_u = "3.14" limit_v = "0.5"
   />
   <cylinder_link
-    name="link1"
-    origin_rpy="0 0 0" origin_xyz="0 0 ${L1/2}"
-    radius="0.35" length="${L1}"
+    name = "link1"
+    origin_rpy = "0 0 0" origin_xyz = "0 0 ${L1/2}"
+    radius = "0.35" length = "${L1}"
     mass = "4"
     ixx = "3" ixy = "0"   ixz = "0"
@@ -37,15 +43,15 @@
   />
   <revolute_joint
-    name="q2" type="revolute"
-    axis_xyz="0 1 0"
-    origin_rpy="0 0 0" origin_xyz="0 0 ${L1}"
-    parent="link1"
-    child="link2"
-    limit_e="1000.0" limit_l="-3.14" limit_u="3.14" limit_v="0.5"
+    name = "q2" type = "revolute"
+    axis_xyz = "0 1 0"
+    origin_rpy = "0 0 0" origin_xyz = "0 0 ${L1}"
+    parent = "link1"
+    child = "link2"
+    limit_e = "1000.0" limit_l = "-3.14" limit_u = "3.14" limit_v = "0.5"
   />
   <cylinder_link
-    name="link2"
-    origin_rpy="0 0 0" origin_xyz="0 0 ${L2/2}"
-    radius="0.15" length="${L2}"
+    name = "link2"
+    origin_rpy = "0 0 0" origin_xyz = "0 0 ${L2/2}"
+    radius = "0.15" length = "${L2}"
     mass = "6"
     ixx = "5" ixy = "0"   ixz = "0"
@@ -54,15 +60,15 @@
   />
   <revolute_joint
-    name="q3" type="revolute"
-    axis_xyz="0 1 0"
-    origin_rpy="0 0 0" origin_xyz="0 0 ${L2}"
-    parent="link2"
-    child="link3"
-    limit_e="1000.0" limit_l="-3.14" limit_u="3.14" limit_v="0.5"
+    name = "q3" type = "revolute"
+    axis_xyz = "0 1 0"
+    origin_rpy = "0 0 0" origin_xyz = "0 0 ${L2}"
+    parent = "link2"
+    child = "link3"
+    limit_e = "1000.0" limit_l = "-3.14" limit_u = "3.14" limit_v = "0.5"
   />
   <cylinder_link
-    name="link3"
-    origin_rpy="0 0 0" origin_xyz="0 0 ${L3/2}"
-    radius="0.15" length="${L3}"
+    name = "link3"
+    origin_rpy = "0 0 0" origin_xyz = "0 0 ${L3/2}"
+    radius = "0.15" length = "${L3}"
     mass = "8"
     ixx = "6" ixy = "0"   ixz = "0"
@@ -70,3 +76,9 @@
                           izz = "6"
   />
+  <!-- End robot description -->
+  <!-- Gazebo node for ros control -->
+  <gazebo>
+    <plugin name="gazebo_ros_control" filename="libgazebo_ros_control.so">
+    </plugin>
+  </gazebo>
 </robot>
